File: PCB files/kicad project/kurako_40.sch (KiCad schematic (older format))
At the start: 108 parts, among them J1 conn, P1 USB_C_Plug_USB2.0, SW1 TAB, SW10 S, SW11 X, SW12 PROG, SW13 E, SW14 D, SW15 C, SW16 ALT, SW17 R, SW18 F, SW19 V, SW2 ESC, SW20 SPACE, SW21 T, SW22 G, SW23 B, SW24 Y, SW25 H, SW26 N, SW27 LOWER, SW28 U, SW29 J, SW3 SHIFT, SW30 M, SW31 RAISE, SW32 I, SW33 K, SW34 ,, SW35 /, SW36 O, SW37 L, SW38 ., SW39 LEFT, SW4 CTRL, SW40 P, SW41 ;, SW42 UP, SW43 DOWN, SW44 BKSP, SW45 ', SW46 ENTER, SW47 RIGHT, SW48 SW_SPST, SW5 Q, SW6 A, SW7 Z, SW8 WIN, SW9 W, U1 ATmega32U4-AU, Y1 16 Mhz

Commit message: bad keyswitch placements
prior rev had bad switch placement, updated and gave the board a rev number
Other:
- note added: "TODO:\n\nSwap Diode package from SOD323 to SOD80\ncorrect RESET switch placement"
Changed lines of the file:
@@
 	8450 2450 8450 2500
 Connection ~ 8450 2450
+Text Notes 500  800  0    50   ~ 0
+TODO:\n\nSwap Diode package from SOD323 to SOD80\ncorrect RESET switch placement
 $EndSCHEMATC

Commit message: board rev changes v1.2
updated schematic from SOD323 diodes to SOD80 due to cost savings and ease of soldering. added ground fill on top and bottom
Parts:
- D1, D10, D11, D12, D13, D14, D15, D16, D17, D18, D19, D2, D20, D21, D22, D23, D24, D25, D26, D27, D28, D29, D3, D30, D31, D32, D33, D34, D35, D36, D37, D38, D39, D4, D40, D41, D42, D43, D44, D45, D46, D47, D5, D6, D7, D8, D9: footprint Diode_SMD:D_SOD-323_HandSoldering -> Diode_SMD:D_MiniMELF

Commit message: minor board and code change
updated usb placement to not stick out as much (-0.75mm)
swapped diode polarity in firmware config
corrected main board header file
Other:
- note removed: "TODO:\n\nSwap Diode package from SOD323 to SOD80\ncorrect RESET switch placement"
Changed lines of the file:
@@
 	8450 2450 8450 2500
 Connection ~ 8450 2450
-Text Notes 500  800  0    50   ~ 0
-TODO:\n\nSwap Diode package from SOD323 to SOD80\ncorrect RESET switch placement
 $EndSCHEMATC

Commit message: usb c updates
chose better USB connector for hand soldering
Parts:
- P1: footprint Connector_USB:USB_C_Receptacle_Amphenol_12401610E4-2A -> 12402012E212A_USB-C:AMPHENOL_12402012E212A; symbol Connector:USB_C_Receptacle_USB2.0 -> 12402012E212A:12402012E212A
Connections:
- net +5V: now also P1.A4_B9 (VBUS), P1.B4_A9 (VBUS__1); no longer P1.A4 (VBUS), P1.A9 (VBUS), P1.B4 (VBUS), P1.B9 (VBUS)
- net GND: now also P1.A1_B12 (GND), P1.B1_A12 (GND__1); no longer P1.A1 (GND), P1.A12 (GND), P1.B1 (GND), P1.B12 (GND), P1.S1 (SHIELD)
- net D1+: now reaches P1.A6 (D+_A), P1.B6 (D+_B), R1.1
- net D1-: now reaches P1.A7 (D-_A), P1.B7 (D-_B), R2.1
Other:
- moved on the sheet: C1, C2, C3, C4, C5, R1, R2, R4, Y1
